File: JoynerX.kicad_pcb (KiCad board)
At the start: 2 copper layers, 33.5 x 42.2 mm, 12 parts, among them J1 USB-AF-DIP-154-HW-S_P1, J2 USB-AF-DIP-154-HW-S_P2, J3 DE9_Plug, J6 no impl., SW1 SW_Push, U1 CH559L

Commit message: rev2 pcb
Parts:
- added C5: 0.1u, Capacitor_SMD:C_0402_1005Metric, F.Cu at (33.9, 43.9)
- added C6: 0.1u, Capacitor_SMD:C_0402_1005Metric, F.Cu at (33.9, 35.6)
- added U2: 74LS257, Package_SO:TSSOP-16_4.4x5mm_P0.65mm, F.Cu at (31.0, 47.3)
- added U3: 74LS257, Package_SO:TSSOP-16_4.4x5mm_P0.65mm, F.Cu at (31.0, 39.1)
- C1, C2, C3, C4: footprint Capacitor_SMD:C_0603_1608Metric_Pad1.08x0.95mm_HandSolder -> Capacitor_SMD:C_0402_1005Metric
- R1: footprint Resistor_SMD:R_0603_1608Metric_Pad0.98x0.95mm_HandSolder -> Resistor_SMD:R_0402_1005Metric
- moved SW1 218.3 mm to (21.6, 42.9), turned to 90 degrees
- moved J2 214.7 mm to (40.6, 55.9)
- moved J3 214.7 mm to (27.0, 33.2)
- moved J1 214.7 mm to (24.5, 55.9)
- moved C3 214.5 mm to (20.5, 50.6), turned to 180 degrees
- moved C4 213.4 mm to (36.8, 50.6)
- moved D1 210.8 mm to (47.3, 47.6), turned to 180 degrees
- moved C2 210.5 mm to (43.8, 46.1)
- moved U1 209.5 mm to (43.2, 40.5)
- moved R1 209.4 mm to (48.3, 48.9)
- moved C1 209.0 mm to (41.9, 46.1)
- moved J6 201.1 mm to (41.0, 49.4), turned to 0 degrees
Connections:
- U1 pad 10: unconnected-(U1-P3_4-Pad10) -> /B6
- U1 pad 11: unconnected-(U1-P3_5-Pad11) -> /B5
- U1 pad 12: unconnected-(U1-P3_6-Pad12) -> /B4
- U1 pad 13: unconnected-(U1-P3_7-Pad13) -> /B3
- U1 pad 15: unconnected-(U1-P4_2-Pad15) -> /OE
- U1 pad 19: unconnected-(U1-P4_1-Pad19) -> /START
- U1 pad 20: unconnected-(U1-P4_0-Pad20) -> /SELECT
- U1 pad 21: /JOY_U -> /B2
- U1 pad 22: /JOY_D -> /B1
- U1 pad 23: /JOY_L -> /RIGHT
- U1 pad 24: /JOY_R -> /LEFT
- U1 pad 25: /JOY_B1 -> /DOWN
- U1 pad 26: /JOY_B2 -> /UP
- U1 pad 27: /JOY_COM -> unconnected-(U1-P2_6-Pad27)
- U1 pad 3: unconnected-(U1-RST-Pad3) -> /JOY_COM
- U1 pad 47: unconnected-(U1-P1_4-Pad47) -> /JOY_COM
Routing:
- net /JOY_COM: track 9.75 -> 79.9 mm, vias 0 -> 3
- net /B5: track 0.00 -> 61.9 mm, vias 0 -> 2
- net GND: track 93.4 -> 153.1 mm, vias 2 -> 1
- net /B6: track 0.00 -> 54.1 mm, vias 0 -> 2
- net /START: track 0.00 -> 51.9 mm, vias 0 -> 2
- net /B2: track 0.00 -> 47.9 mm, vias 0 -> 2
- net /OE: track 0.00 -> 36.0 mm, vias 0 -> 3
- net /B4: track 0.00 -> 34.1 mm, vias 0 -> 2
- net /BTN: track 22.8 -> 52.2 mm, vias 0 -> 2
- net /B1: track 0.00 -> 28.7 mm, vias 0 -> 2
- net /H1_D-: track 15.8 -> 40.2 mm
- net /B3: track 0.00 -> 17.6 mm
- net /UP: track 0.00 -> 13.4 mm, vias 0 -> 2
- net /JOY_B1: track 10.0 -> 22.6 mm
- net /DOWN: track 0.00 -> 12.4 mm, vias 0 -> 2
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Other:
- board size 33.5 x 42.2 mm -> 33.7 x 40 mm
- board text added: "+"
- board text added: "2023.10.22 Rev.2 Designed By Mellow PCB MP17-MOONSHOT"
- board text added: "MP17"
- board text added: "Moonshot"
- board text added: "TX"
- board text added: "by Mellow PCB"
