File: JoynerX.kicad_sch (KiCad schematic)
At the start: 12 parts, among them J1 USB-AF-DIP-154-HW-S_P1, J2 USB-AF-DIP-154-HW-S_P2, J3 DE9_Plug, J6 no impl., SW1 SW_Push, U1 CH559L

Commit message: rev2 pcb
Parts:
- added C5, C6: 0.1u, Capacitor_SMD:C_0402_1005Metric, symbol Device:C
- added U2, U3: 74LS257, Package_SO:TSSOP-16_4.4x5mm_P0.65mm, symbol 74xx:74LS257
- C1, C2, C3, C4: footprint Capacitor_SMD:C_0603_1608Metric_Pad1.08x0.95mm_HandSolder -> Capacitor_SMD:C_0402_1005Metric
- R1: footprint Resistor_SMD:R_0603_1608Metric_Pad0.98x0.95mm_HandSolder -> Resistor_SMD:R_0402_1005Metric
Connections:
- net GND: now also C5.2, C6.2, U2.2 (I0a), U2.3 (I1a), U2.5 (I0b), U2.6 (I1b), U2.8 (GND), U3.8 (GND)
- net JOY_B1: now also U2.9 (Zd); no longer U1.25 (P2_4)
- net JOY_B2: now also U3.7 (Zb); no longer U1.26 (P2_5)
- net JOY_COM: now also U1.3 (RST), U1.47 (P1_4), U2.1 (S), U3.1 (S); no longer U1.27 (P2_6)
- net JOY_D: now also U3.4 (Za); no longer U1.22 (P2_1)
- net JOY_L: now also U3.9 (Zd); no longer U1.23 (P2_2)
- net JOY_R: now also U3.12 (Zc); no longer U1.24 (P2_3)
- net JOY_U: now also U2.12 (Zc); no longer U1.21 (P2_0)
- net VCC: now also C5.1, C6.1, U2.16 (VCC), U3.16 (VCC)
- net B6: now reaches U1.10 (P3_4)
- net B6: now also U2.10 (I1d)
- net B5: now reaches U1.11 (P3_5)
- net B5: now also U3.6 (I1b)
- net B4: now reaches U1.12 (P3_6)
- net B4: now also U3.13 (I1c)
- net B3: now reaches U1.13 (P3_7)
- net B3: now also U2.13 (I1c)
- net OE: now reaches U1.15 (P4_2)
- net OE: now also U2.15 (OE), U3.15 (OE)
- net START: now reaches U1.19 (P4_1)
- net START: now also U3.3 (I1a)
- net SELECT: now reaches U1.20 (P4_0)
- net SELECT: now also U3.10 (I1d)
- new net B1: U1.22 (P2_1), U2.14 (I0c)
- new net B2: U1.21 (P2_0), U3.2 (I0a)
- new net DOWN: U1.25 (P2_4), U3.5 (I0b)
- new net LEFT: U1.24 (P2_3), U3.14 (I0c)
- new net RIGHT: U1.23 (P2_2), U3.11 (I0d)
- new net UP: U1.26 (P2_5), U2.11 (I0d)
- no-connect marks 33 -> 27
