File: KiCAD/Moonshot.kicad_sch (KiCad schematic)
At the start: 16 parts, among them J1 USB-AF-DIP-154-HW-S_P1, J2 USB-AF-DIP-154-HW-S_P2, J3 DE9_Plug, J6 no impl., SW1 SW_Push, U1 CH559L, U2 74LS257, U3 74LS257

Commit message: v3 pcb
Parts:
- added J4: HY2.0-4P, toyoshim:CONN-TH_4P-P2.00_HX20020-4A_2, symbol Connector_Generic:Conn_01x04
Connections:
- net GND: now also J4.1 (Pin_1)
- net VCC: now also J4.2 (Pin_2)
- net SDA: now reaches U1.38 (P0_2)
- net SDA: now also U1.43 (P1_0), J4.3 (Pin_3)
- net SCL: now reaches U1.39 (P0_1)
- net SCL: now also J4.4 (Pin_4)
- no-connect marks 27 -> 24

Commit message: Rev.5 board
Parts:
- added R2, R3: 1k, Resistor_SMD:R_0402_1005Metric, symbol Device:R
Connections:
- net JOY_B1: now also R2.2; no longer U2.9 (Zd)
- net JOY_B2: now also R3.2; no longer U3.7 (Zb)
- new net: R3.1, U3.7 (Zb)
- new net: R2.1, U2.9 (Zd)
Changed lines of the file:
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@@
     (stroke (width 0) (type default))
   )
-  (wire (pts (xy 90.17 149.86) (xy 99.06 149.86))
+  (wire (pts (xy 97.79 149.86) (xy 106.68 149.86))
     (stroke (width 0) (type default))
   )
@@
     (stroke (width 0) (type default))
   )
-  (wire (pts (xy 149.225 134.62) (xy 158.115 134.62))
+  (wire (pts (xy 156.845 134.62) (xy 165.735 134.62))
     (stroke (width 0) (type default))
   )
@@
     (effects (font (size 1.27 1.27)) (justify left bottom))
   )
-  (label "JOY_B1" (at 90.805 149.86 0) (fields_autoplaced)
+  (label "JOY_B1" (at 98.425 149.86 0) (fields_autoplaced)
     (effects (font (size 1.27 1.27)) (justify left bottom))
   )
@@
     (effects (font (size 1.27 1.27)) (justify left bottom))
   )
-  (label "JOY_B2" (at 149.86 134.62 0) (fields_autoplaced)
+  (label "JOY_B2" (at 157.48 134.62 0) (fields_autoplaced)
     (effects (font (size 1.27 1.27)) (justify left bottom))
   )
@@
         (path "/18d2f8f4-5c79-4049-a93f-1d89af805da9"
           (reference "#PWR021") (unit 1)
+        )
+      )
+    )
+  )
+  (symbol (lib_id "Device:R") (at 153.035 134.62 90) (unit 1)
+    (in_bom yes) (on_board yes) (dnp no) (fields_autoplaced)
+    (property "Reference" "R3" (at 153.035 130.5941 90)
+      (effects (font (size 1.27 1.27)))
+    )
+    (property "Value" "1k" (at 153.035 132.5151 90)
+      (effects (font (size 1.27 1.27)))
+    )
+    (property "Footprint" "Resistor_SMD:R_0402_1005Metric" (at 153.035 136.398 90)
+      (effects (font (size 1.27 1.27)) hide)
+    )
+    (property "Datasheet" "~" (at 153.035 134.62 0)
+      (effects (font (size 1.27 1.27)) hide)
+    )
+    (pin "1")
+    (pin "2")
+    (instances
+      (project "Moonshot"
+        (path "/18d2f8f4-5c79-4049-a93f-1d89af805da9"
+          (reference "R3") (unit 1)
         )
       )
@@
         )
       )
+    )
+  )
+  (symbol (lib_id "Device:R") (at 93.98 149.86 90) (unit 1)
+    (in_bom yes) (on_board yes) (dnp no) (fields_autoplaced)
+    (property "Reference" "R2" (at 93.98 145.8341 90)
+      (effects (font (size 1.27 1.27)))
+    )
+    (property "Value" "1k" (at 93.98 147.7551 90)
+      (effects (font (size 1.27 1.27)))
+    )
+    (property "Footprint" "Resistor_SMD:R_0402_1005Metric" (at 93.98 151.638 90)
+      (effects (font (size 1.27 1.27)) hide)
+    )
+    (property "Datasheet" "~" (at 93.98 149.86 0)
+      (effects (font (size 1.27 1.27)) hide)
+    )
+    (pin "1")
+    (pin "2")
+    (instances
+      (project "Moonshot"
+        (path "/18d2f8f4-5c79-4049-a93f-1d89af805da9"
+          (reference "R2") (unit 1)
+        )
+      )

Commit message: PCB Rev.7
Parts:
- R2, R3: value 1k -> 100
Connections:
- net B1: now also U1.26 (P2_5), U2.11 (I0d); no longer U1.22 (P2_1), U2.14 (I0c)
- net B2: now also U1.25 (P2_4), U3.5 (I0b); no longer U1.21 (P2_0), U3.2 (I0a)
- net B3: now also U1.10 (P3_4), U2.10 (I1d); no longer U1.13 (P3_7), U2.13 (I1c)
- net B4: now also U1.20 (P4_0), U3.10 (I1d); no longer U1.12 (P3_6), U3.13 (I1c)
- net B5: now also U1.19 (P4_1), U3.3 (I1a); no longer U1.11 (P3_5), U3.6 (I1b)
- net B6: now also U1.13 (P3_7), U2.13 (I1c); no longer U1.10 (P3_4), U2.10 (I1d)
- net DOWN: now also U1.21 (P2_0), U3.2 (I0a); no longer U1.25 (P2_4), U3.5 (I0b)
- net LEFT: now also U1.23 (P2_2), U3.11 (I0d); no longer U1.24 (P2_3), U3.14 (I0c)
- net RIGHT: now also U1.24 (P2_3), U3.14 (I0c); no longer U1.23 (P2_2), U3.11 (I0d)
- net SELECT: now also U1.12 (P3_6), U3.13 (I1c); no longer U1.20 (P4_0), U3.10 (I1d)
- net START: now also U1.11 (P3_5), U3.6 (I1b); no longer U1.19 (P4_1), U3.3 (I1a)
- net UP: now also U1.22 (P2_1), U2.14 (I0c); no longer U1.26 (P2_5), U2.11 (I0d)
Changed lines of the file:
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@@
     (effects (font (size 1.27 1.27)) (justify left bottom))
   )
-  (label "B5" (at 115.57 137.16 0) (fields_autoplaced)
-    (effects (font (size 1.27 1.27)) (justify left bottom))
-  )
-  (label "UP" (at 56.515 149.86 0) (fields_autoplaced)
+  (label "B5" (at 115.6208 129.54 0) (fields_autoplaced)
+    (effects (font (size 1.27 1.27)) (justify left bottom))
+  )
+  (label "UP" (at 56.515 142.24 0) (fields_autoplaced)
     (effects (font (size 1.27 1.27)) (justify left bottom))
   )
@@
     (effects (font (size 1.27 1.27)) (justify left bottom))
   )
-  (label "START" (at 55.88 90.17 0) (fields_autoplaced)
+  (label "START" (at 56.388 67.31 0) (fields_autoplaced)
     (effects (font (size 1.27 1.27)) (justify left bottom))
   )
@@
     (effects (font (size 1.27 1.27)) (justify left bottom))
   )
-  (label "RIGHT" (at 55.88 100.33 0) (fields_autoplaced)
-    (effects (font (size 1.27 1.27)) (justify left bottom))
-  )
-  (label "RIGHT" (at 115.57 149.86 0) (fields_autoplaced)
+  (label "RIGHT" (at 55.88 102.87 0) (fields_autoplaced)
+    (effects (font (size 1.27 1.27)) (justify left bottom))
+  )
+  (label "RIGHT" (at 115.57 142.24 0) (fields_autoplaced)
     (effects (font (size 1.27 1.27)) (justify left bottom))
   )
@@
     (effects (font (size 1.27 1.27)) (justify left bottom))
   )
-  (label "SELECT" (at 55.88 92.71 0) (fields_autoplaced)
+  (label "SELECT" (at 56.134 69.85 0) (fields_autoplaced)
     (effects (font (size 1.27 1.27)) (justify left bottom))
   )
@@
     (effects (font (size 1.27 1.27)) (justify left bottom))
   )
-  (label "B2" (at 55.88 95.25 0) (fields_autoplaced)
-    (effects (font (size 1.27 1.27)) (justify left bottom))
-  )
-  (label "B2" (at 115.57 127 0) (fields_autoplaced)
+  (label "B2" (at 90.678 102.87 0) (fields_autoplaced)
+    (effects (font (size 1.27 1.27)) (justify left bottom))
+  )
+  (label "B2" (at 115.57 134.62 0) (fields_autoplaced)
     (effects (font (size 1.27 1.27)) (justify left bottom))
   )
@@
     (effects (font (size 1.27 1.27)) (justify left bottom))
   )
-  (label "B5" (at 55.88 67.31 0) (fields_autoplaced)
-    (effects (font (size 1.27 1.27)) (justify left bottom))
-  )
-  (label "DOWN" (at 115.57 134.62 0) (fields_autoplaced)
+  (label "B5" (at 55.88 90.17 0) (fields_autoplaced)
+    (effects (font (size 1.27 1.27)) (justify left bottom))
+  )
+  (label "DOWN" (at 115.6208 127 0) (fields_autoplaced)
     (effects (font (size 1.27 1.27)) (justify left bottom))
   )
@@
     (effects (font (size 1.27 1.27)) (justify left bottom))
   )
-  (label "SELECT" (at 115.57 152.4 0) (fields_autoplaced)
+  (label "SELECT" (at 115.57 144.78 0) (fields_autoplaced)
     (effects (font (size 1.27 1.27)) (justify left bottom))
   )
@@
     (effects (font (size 1.27 1.27)) (justify left bottom))
   )
-  (label "START" (at 115.57 129.54 0) (fields_autoplaced)
+  (label "START" (at 115.57 137.16 0) (fields_autoplaced)
     (effects (font (size 1.27 1.27)) (justify left bottom))
   )
@@
     (effects (font (size 1.27 1.27)) (justify left bottom))
   )
-  (label "LEFT" (at 115.57 142.24 0) (fields_autoplaced)
+  (label "LEFT" (at 115.824 149.86 0) (fields_autoplaced)
     (effects (font (size 1.27 1.27)) (justify left bottom))
   )
@@
     (effects (font (size 1.27 1.27)) (justify left bottom))
   )
-  (label "B4" (at 115.57 144.78 0) (fields_autoplaced)
-    (effects (font (size 1.27 1.27)) (justify left bottom))
-  )
-  (label "UP" (at 90.805 100.33 0) (fields_autoplaced)
-    (effects (font (size 1.27 1.27)) (justify left bottom))
-  )
-  (label "B1" (at 55.88 97.79 0) (fields_autoplaced)
+  (label "B4" (at 115.824 152.4 0) (fields_autoplaced)
+    (effects (font (size 1.27 1.27)) (justify left bottom))
+  )
+  (label "UP" (at 56.007 97.79 0) (fields_autoplaced)
+    (effects (font (size 1.27 1.27)) (justify left bottom))
+  )
+  (label "B1" (at 90.678 100.33 0) (fields_autoplaced)
     (effects (font (size 1.27 1.27)) (justify left bottom))
   )
@@
     (effects (font (size 1.27 1.27)) (justify left bottom))
   )
-  (label "B6" (at 55.88 64.77 0) (fields_autoplaced)
-    (effects (font (size 1.27 1.27)) (justify left bottom))
-  )
-  (label "B1" (at 56.515 142.24 0) (fields_autoplaced)
+  (label "B6" (at 56.388 74.93 0) (fields_autoplaced)
+    (effects (font (size 1.27 1.27)) (justify left bottom))
+  )
+  (label "B1" (at 56.515 149.86 0) (fields_autoplaced)
     (effects (font (size 1.27 1.27)) (justify left bottom))
   )
@@
     (effects (font (size 1.27 1.27)) (justify left bottom))
   )
-  (label "B3" (at 56.515 144.78 0) (fields_autoplaced)
+  (label "B3" (at 56.515 152.4 0) (fields_autoplaced)
     (effects (font (size 1.27 1.27)) (justify left bottom))
   )
@@
     (effects (font (size 1.27 1.27)) (justify left bottom))
   )
-  (label "LEFT" (at 55.88 102.87 0) (fields_autoplaced)
-    (effects (font (size 1.27 1.27)) (justify left bottom))
-  )
-  (label "B6" (at 56.515 152.4 0) (fields_autoplaced)
+  (label "LEFT" (at 55.88 100.33 0) (fields_autoplaced)
+    (effects (font (size 1.27 1.27)) (justify left bottom))
+  )
+  (label "B6" (at 56.515 144.78 0) (fields_autoplaced)
     (effects (font (size 1.27 1.27)) (justify left bottom))
   )
@@
     (effects (font (size 1.27 1.27)) (justify left bottom))
   )
-  (label "B3" (at 55.88 74.93 0) (fields_autoplaced)
+  (label "B3" (at 56.388 64.77 0) (fields_autoplaced)
     (effects (font (size 1.27 1.27)) (justify left bottom))
   )
@@
     (effects (font (size 1.27 1.27)) (justify left bottom))
   )
-  (label "DOWN" (at 90.805 102.87 0) (fields_autoplaced)
-    (effects (font (size 1.27 1.27)) (justify left bottom))
-  )
-  (label "B4" (at 55.88 69.85 0) (fields_autoplaced)
+  (label "DOWN" (at 55.88 95.25 0) (fields_autoplaced)
+    (effects (font (size 1.27 1.27)) (justify left bottom))
+  )
+  (label "B4" (at 55.88 92.71 0) (fields_autoplaced)
     (effects (font (size 1.27 1.27)) (justify left bottom))
   )
@@
       (effects (font (size 1.27 1.27)))
     )
-    (property "Value" "1k" (at 153.035 132.5151 90)
+    (property "Value" "100" (at 153.035 132.5151 90)
       (effects (font (size 1.27 1.27)))
     )
@@
       (effects (font (size 1.27 1.27)))
     )
-    (property "Value" "1k" (at 93.98 147.7551 90)
-      (effects (font (size 1.27 1.27)))
-    )
+    (property "Value" "100" (at 93.98 147.7551 90)
+      (effects (font (size 1.27 1.27)))
+    )
